File: hardware/linear-poti-v2.kicad_pcb (KiCad board)
At the start: 2 copper layers, 85 x 25 mm, 22 parts, among them P1 CON-SENSOR2, P2 DEBUG, P3 BOOT, U1 XMC1XXX24, U3 DRILL, U4 DRILL, U5 DRILL, U6 DRILL

Commit message: Fix page settings
Other:
- board text added: "Copyright Tinkerforge GmbH 2018. This documentation describes Open Hardware and is licensed under the CERN OHL v. 1.1. You may redistribute and modify this documentation under the terms of the CERN OHL v.1.1. (http://ohwr.org/cernohl). This documentation is distributed WITHOUT ANY EXPRESS OR IMPLIED WARRANTY, INCLUDING OF MERCHANTABILITY, SATISFACTORY QUALITY AND FITNESS FOR A PARTICULAR PURPOSE.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"
- board text removed: "Copyright Tinkerforge GmbH 2011. This documentation describes Open Hardware and is licensed under the CERN OHL v. 1.1. You may redistribute and modify this documentation under the terms of the CERN OHL v.1.1. (http://ohwr.org/cernohl). This documentation is distributed WITHOUT ANY EXPRESS OR IMPLIED WARRANTY, INCLUDING OF MERCHANTABILITY, SATISFACTORY QUALITY AND FITNESS FOR A PARTICULAR PURPOSE.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"
Changed lines of the file:
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@@
     (links 36)
     (no_connects 0)
-    (area 109.309499 66.309499 194.690501 91.690501)
+    (area 108.644999 65.644999 283.02204 165.61816)
     (thickness 1.6002)
     (drawings 12)
@@
   (title_block
     (title "Linear Poti Bricklet")
-    (date 2016-03-04)
-    (rev 1.2)
+    (date 2018-06-22)
+    (rev 2.0)
     (company "Tinkerforge GmbH")
     (comment 1 "Licensed under CERN OHL v.1.1")
-    (comment 2 "Copyright (©) 2016, B.Nordmeyer <bastian@tinkerforge.com>")
+    (comment 2 "Copyright (©) 2018, L.Lauer <lukas@tinkerforge.com>")
   )
   (layers
@@
   )
   (setup
-    (last_trace_width 0.25)
+    (last_trace_width 0.2)
     (user_trace_width 0.2)
     (user_trace_width 0.25)
@@
   (gr_arc (start 112 89) (end 112 91.5) (angle 90) (layer Edge.Cuts) (width 0.381))
   (gr_arc (start 192 69) (end 192 66.5) (angle 90) (layer Edge.Cuts) (width 0.381))
-  (gr_text "Copyright Tinkerforge GmbH 2011.\nThis documentation describes Open Hardware and is licensed under the\nCERN OHL v. 1.1.\nYou may redistribute and modify this documentation under the terms of the\nCERN OHL v.1.1. (http://ohwr.org/cernohl). This documentation is distributed\nWITHOUT ANY EXPRESS OR IMPLIED WARRANTY, INCLUDING OF\nMERCHANTABILITY, SATISFACTORY QUALITY AND FITNESS FOR A\nPARTICULAR PURPOSE. Please see the CERN OHL v.1.1 for applicable\nconditions" (at 258.97586 159.67456) (layer Cmts.User)
-    (effects (font (size 0.8001 0.8001) (thickness 0.20066)))
+  (gr_text "Copyright Tinkerforge GmbH 2018.\nThis documentation describes Open Hardware and is licensed under the\nCERN OHL v. 1.1.\nYou may redistribute and modify this documentation under the terms of the\nCERN OHL v.1.1. (http://ohwr.org/cernohl). This documentation is distributed\nWITHOUT ANY EXPRESS OR IMPLIED WARRANTY, INCLUDING OF\nMERCHANTABILITY, SATISFACTORY QUALITY AND FITNESS FOR A\nPARTICULAR PURPOSE. Please see the CERN OHL v.1.1 for applicable\nconditions" (at 258.97586 159.67456) (layer Cmts.User)
+    (effects (font (size 0.8001 0.8001) (thickness 0.200025)))
   )
   (gr_text tinkerforge.com (at 129.30124 87.5538) (layer F.SilkS)

Commit message: Fix pin of IN_1
Connections:
- U1 pad 18: IN_1 -> Net-(U1-Pad18)
- U1 pad 2: Net-(U1-Pad2) -> IN_1
Routing:
- net IN_1: track 6.41 -> 13.4 mm, vias 0 -> 1
- net Net-(U1-Pad18): track 0.00 -> 0.64 mm
Changed lines of the file:
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@@
     (links 36)
     (no_connects 0)
-    (area 108.644999 65.644999 283.02204 165.61816)
+    (area 109.309499 66.309499 194.690501 91.690501)
     (thickness 1.6002)
     (drawings 12)
-    (tracks 119)
+    (tracks 123)
     (zones 0)
     (modules 22)
@@
   (net 15 S-CLK)
   (net 16 S-CS)
-  (net 17 "Net-(U1-Pad2)")
-  (net 18 "Net-(U1-Pad3)")
-  (net 19 "Net-(U1-Pad5)")
-  (net 20 "Net-(U1-Pad6)")
-  (net 21 "Net-(U1-Pad8)")
-  (net 22 "Net-(U1-Pad11)")
-  (net 23 "Net-(U1-Pad12)")
-  (net 24 "Net-(U1-Pad14)")
-  (net 25 "Net-(U1-Pad16)")
-  (net 26 "Net-(U1-Pad19)")
-  (net 27 "Net-(U1-Pad20)")
-  (net 28 "Net-(U1-Pad21)")
-  (net 29 "Net-(U1-Pad7)")
-  (net 30 "Net-(U1-Pad4)")
+  (net 17 "Net-(U1-Pad3)")
+  (net 18 "Net-(U1-Pad5)")
+  (net 19 "Net-(U1-Pad6)")
+  (net 20 "Net-(U1-Pad8)")
+  (net 21 "Net-(U1-Pad11)")
+  (net 22 "Net-(U1-Pad12)")
+  (net 23 "Net-(U1-Pad14)")
+  (net 24 "Net-(U1-Pad16)")
+  (net 25 "Net-(U1-Pad19)")
+  (net 26 "Net-(U1-Pad20)")
+  (net 27 "Net-(U1-Pad21)")
+  (net 28 "Net-(U1-Pad7)")
+  (net 29 "Net-(U1-Pad4)")
+  (net 30 "Net-(U1-Pad18)")
   (net_class Default "Dies ist die voreingestellte Netzklasse."
     (clearance 0.15)
@@
     (add_net "Net-(U1-Pad14)")
     (add_net "Net-(U1-Pad16)")
+    (add_net "Net-(U1-Pad18)")
     (add_net "Net-(U1-Pad19)")
-    (add_net "Net-(U1-Pad2)")
     (add_net "Net-(U1-Pad20)")
     (add_net "Net-(U1-Pad21)")
@@
       (net 13 S-MISO))
     (pad 2 smd oval (at -2.025 -0.75 180) (size 1 0.3) (layers Vorderseite F.Paste F.Mask)
-      (net 17 "Net-(U1-Pad2)"))
+      (net 2 IN_1))
     (pad 3 smd oval (at -2.025 -0.25 180) (size 1 0.3) (layers Vorderseite F.Paste F.Mask)
-      (net 18 "Net-(U1-Pad3)"))
+      (net 17 "Net-(U1-Pad3)"))
     (pad 4 smd oval (at -2.025 0.25 180) (size 1 0.3) (layers Vorderseite F.Paste F.Mask)
-      (net 30 "Net-(U1-Pad4)"))
+      (net 29 "Net-(U1-Pad4)"))
     (pad 5 smd oval (at -2.025 0.75 180) (size 1 0.3) (layers Vorderseite F.Paste F.Mask)
-      (net 19 "Net-(U1-Pad5)"))
+      (net 18 "Net-(U1-Pad5)"))
     (pad 6 smd oval (at -2.025 1.25 180) (size 1 0.3) (layers Vorderseite F.Paste F.Mask)
-      (net 20 "Net-(U1-Pad6)"))
+      (net 19 "Net-(U1-Pad6)"))
     (pad 7 smd oval (at -1.25 2.025 270) (size 1 0.3) (layers Vorderseite F.Paste F.Mask)
-      (net 29 "Net-(U1-Pad7)"))
+      (net 28 "Net-(U1-Pad7)"))
     (pad 8 smd oval (at -0.75 2.025 270) (size 1 0.3) (layers Vorderseite F.Paste F.Mask)
-      (net 21 "Net-(U1-Pad8)"))
+      (net 20 "Net-(U1-Pad8)"))
     (pad 9 smd oval (at -0.25 2.025 270) (size 1 0.3) (layers Vorderseite F.Paste F.Mask)
       (net 1 GND))
@@
       (net 3 VCC))
     (pad 11 smd oval (at 0.75 2.025 270) (size 1 0.3) (layers Vorderseite F.Paste F.Mask)
-      (net 22 "Net-(U1-Pad11)"))
+      (net 21 "Net-(U1-Pad11)"))
     (pad 12 smd oval (at 1.25 2.025 270) (size 1 0.3) (layers Vorderseite F.Paste F.Mask)
-      (net 23 "Net-(U1-Pad12)"))
+      (net 22 "Net-(U1-Pad12)"))
     (pad 13 smd oval (at 2.025 1.25 180) (size 1 0.3) (layers Vorderseite F.Paste F.Mask)
       (net 12 "Net-(R3-Pad1)"))
     (pad 14 smd oval (at 2.025 0.75 180) (size 1 0.3) (layers Vorderseite F.Paste F.Mask)
-      (net 24 "Net-(U1-Pad14)"))
+      (net 23 "Net-(U1-Pad14)"))
     (pad 15 smd oval (at 2.025 0.25 180) (size 1 0.3) (layers Vorderseite F.Paste F.Mask)
       (net 10 "Net-(P2-Pad1)"))
     (pad 16 smd oval (at 2.025 -0.25 180) (size 1 0.3) (layers Vorderseite F.Paste F.Mask)
-      (net 25 "Net-(U1-Pad16)"))
+      (net 24 "Net-(U1-Pad16)"))
     (pad 17 smd oval (at 2.025 -0.75 180) (size 1 0.3) (layers Vorderseite F.Paste F.Mask)
       (net 11 "Net-(P3-Pad2)"))
     (pad 18 smd oval (at 2.025 -1.25 180) (size 1 0.3) (layers Vorderseite F.Paste F.Mask)
-      (net 2 IN_1))
+      (net 30 "Net-(U1-Pad18)"))
     (pad 19 smd oval (at 1.25 -2.025 270) (size 1 0.3) (layers Vorderseite F.Paste F.Mask)
-      (net 26 "Net-(U1-Pad19)"))
+      (net 25 "Net-(U1-Pad19)"))
     (pad 20 smd oval (at 0.75 -2.025 270) (size 1 0.3) (layers Vorderseite F.Paste F.Mask)
-      (net 27 "Net-(U1-Pad20)"))
+      (net 26 "Net-(U1-Pad20)"))
     (pad 21 smd oval (at 0.25 -2.025 270) (size 1 0.3) (layers Vorderseite F.Paste F.Mask)
-      (net 28 "Net-(U1-Pad21)"))
+      (net 27 "Net-(U1-Pad21)"))
     (pad 22 smd oval (at -0.25 -2.025 270) (size 1 0.3) (layers Vorderseite F.Paste F.Mask)
       (net 16 S-CS))
@@
   (segment (start 193.3 73.1) (end 193.3 74.08) (width 0.55) (layer Vorderseite) (net 1))
   (via (at 193.3 74.08) (size 0.55) (drill 0.2) (layers Vorderseite Rückseite) (net 1))
-  (segment (start 182.575 72.45) (end 181.93 72.45) (width 0.25) (layer Vorderseite) (net 2))
+  (segment (start 184.40112 77.10994) (end 184.40112 75.25888) (width 0.2) (layer Rückseite) (net 2))
+  (segment (start 187.71 71.95) (end 186.625 71.95) (width 0.2) (layer Vorderseite) (net 2))
+  (via (at 187.71 71.95) (size 0.55) (drill 0.2) (layers Vorderseite Rückseite) (net 2))
+  (segment (start 184.40112 75.25888) (end 187.71 71.95) (width 0.2) (layer Rückseite) (net 2))
   (segment (start 181.83 74.53882) (end 184.40112 77.10994) (width 0.25) (layer Vorderseite) (net 2))
   (segment (start 181.83 72.55) (end 181.83 74.53882) (width 0.25) (layer Vorderseite) (net 2))
@@
   (segment (start 185.8393 75.9693) (end 186.545 75.9693) (width 0.2) (layer Vorderseite) (net 16))
   (segment (start 184.85 74.98) (end 185.8393 75.9693) (width 0.2) (layer Vorderseite) (net 16))
+  (segment (start 182.575 72.45) (end 181.93 72.45) (width 0.25) (layer Vorderseite) (net 30))
   (zone (net 1) (net_name GND) (layer Rückseite) (hatch edge 0.508)
     (connect_pads yes (clearance 0.15))
