File: hardware/linear-poti-v2.kicad_pcb (KiCad board)
At the start: 2 copper layers, 85 x 25 mm, 22 parts, among them P1 CON-SENSOR2, P2 DEBUG, P3 BOOT, U1 XMC1XXX24, U3 DRILL, U4 DRILL, U5 DRILL, U6 DRILL

Commit message: remove faulty poti connection, drc
Connections:
- P1 pad 1: Net-(P1-Pad1) -> (no net)
- U1 pad 11: Net-(U1-Pad11) -> (no net)
- U1 pad 12: Net-(U1-Pad12) -> (no net)
- U1 pad 14: Net-(U1-Pad14) -> (no net)
- U1 pad 16: Net-(U1-Pad16) -> (no net)
- U1 pad 18: Net-(U1-Pad18) -> (no net)
- U1 pad 19: Net-(U1-Pad19) -> (no net)
- U1 pad 20: Net-(U1-Pad20) -> (no net)
- U1 pad 21: Net-(U1-Pad21) -> (no net)
- U1 pad 3: Net-(U1-Pad3) -> (no net)
- U1 pad 4: Net-(U1-Pad4) -> (no net)
- U1 pad 5: Net-(U1-Pad5) -> (no net)
- U1 pad 6: Net-(U1-Pad6) -> (no net)
- U1 pad 7: Net-(U1-Pad7) -> (no net)
- U1 pad 8: Net-(U1-Pad8) -> (no net)
Routing:
- net IN_1: track 13.4 -> 7.62 mm
- net Net-(U1-Pad18): track 0.64 -> 0.00 mm

Commit message: changed processor to XMC1100
Parts:
- U1: value XMC1XXX24 -> XMC1100
Changed lines of the file:
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@@
       (effects (font (size 0.3 0.3) (thickness 0.075)))
     )
-    (fp_text value XMC1XXX24 (at 0 0.8 180) (layer F.Fab)
+    (fp_text value XMC1100 (at 0 0.8 180) (layer F.Fab)
       (effects (font (size 0.3 0.3) (thickness 0.075)))
     )
